File: ch32-baseboard-kicad/ch32-baseboard-kicad.kicad_pcb (KiCad board)
At the start: 4 copper layers, 55 x 36 mm, 48 parts, among them J1 USB_C_USB2.0_16P, J2 TC2030, J3 53048-0310, SW1 SW_DIP_x02, SW2 TS-1088, U1 CH32V30xRxTx, U2 SPX3819M5-L-3-3, U3 INA195, X1 16MHz

Commit message: feat: ch32 baseboard v1.1
Parts:
- added R8: 0R, Resistor_SMD:R_0402_1005Metric, F.Cu at (128.8, 133.0)
- C1, C2, C4: value 470n -> 0.1u; footprint Capacitor_SMD:C_0603_1608Metric -> Capacitor_SMD:C_0402_1005Metric
- C13, C14: value 8p -> 10p
- D3: value ESDALC6V1W5 -> ESDALC6V1P6; footprint ch32-baseboard-lib:SOT323-5L-STM -> ch32-baseboard-lib:SOT-666IP-STM
- moved kibuzzard-692C8041 20.5 mm to (98.8, 132.8)
- moved D2 15.3 mm to (101.5, 132.8), turned to 0 degrees
- moved R5 9.76 mm to (104.8, 132.8), turned to 180 degrees
- moved C6 5.18 mm to (119.1, 135.1), turned to 0 degrees
- moved R4 4.18 mm to (115.7, 132.5), turned to -90 degrees
- moved C5 3.69 mm to (113.5, 129.0)
- moved SW2 1.75 mm to (117.0, 125.0)
- moved kibuzzard-692C82FA 1.75 mm to (119.9, 123.6)
- moved C13 1.35 mm to (127.2, 134.6)
- moved C14 1.35 mm to (129.2, 134.6)
- moved X1 1.35 mm to (128.2, 137.0)
- moved D3 1.14 mm to (120.0, 118.0), turned to 0 degrees
- moved C3 0.90 mm to (111.0, 129.0), turned to 90 degrees
- moved C15 0.72 mm to (116.5, 121.3), turned to 180 degrees
- moved J2 0.71 mm to (113.2, 115.0), turned to 180 degrees
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Connections:
- C14 pad 1: /OSC_OUT -> Net-(C14-Pad1)
- D3 pad 5: unconnected-(D3-Pad5) -> GND
- X1 pad 3: /OSC_OUT -> Net-(C14-Pad1)
Routing:
- net /SWDIO: track 31.7 -> 18.4 mm
- net /NRST: track 33.2 -> 43.5 mm, vias 2 -> 3
- net GND: track 19.9 -> 28.2 mm, vias 127 -> 116
- net /SWCLK: track 23.2 -> 16.0 mm
- net +3V3S: track 85.3 -> 89.8 mm, vias 7 -> 6
- net Net-(C14-Pad1): track 0.00 -> 3.44 mm
- net /INA_VOUT: track 17.0 -> 13.7 mm
- net /OSC_OUT: track 5.03 -> 1.92 mm
- net /OSC_IN: track 6.61 -> 7.96 mm
- net +VBUSF: track 10.4 -> 9.55 mm
- net +3V3: track 49.8 -> 49.1 mm, vias 2 -> 6
