File: ch32-baseboard-kicad/ch32-baseboard-kicad.kicad_sch (KiCad schematic)
At the start: 42 parts, among them J1 USB_C_USB2.0_16P, J2 TC2030, J3 53048-0310, SW1 SW_DIP_x02, SW2 TS-1088, U1 CH32V30xRxTx, U2 SPX3819M5-L-3-3, U3 INA195, X1 16MHz

Commit message: feat: ch32 baseboard v1.1
Parts:
- removed D3: ESDALC6V1W5, ch32-baseboard-lib:SOT323-5L-STM, symbol ch32-baseboard-lib:ESDALC6V1W5
- removed J3: 53048-0310, Connector_Molex:Molex_PicoBlade_53048-0310_1x03_P1.25mm_Horizontal, symbol Connector:Conn_01x03_Pin
- added D3: ESDALC6V1P6, ch32-baseboard-lib:SOT-666IP-STM, symbol ch32-baseboard-lib:ESDALC6V1P6
- added J3: 53048-0310, Connector_Molex:Molex_PicoBlade_53048-0310_1x03_P1.25mm_Horizontal, symbol Connector_Generic:Conn_01x03
- added R8: 0R, Resistor_SMD:R_0402_1005Metric, symbol Device:R
- C1, C2, C4: value 470n -> 0.1u; footprint Capacitor_SMD:C_0603_1608Metric -> Capacitor_SMD:C_0402_1005Metric; Manufacturer Samsung Electro-Mechanics -> Samsung; Manufacturer Part Number CL10B474KA8NNNC -> CL05B104KO5NNNC
- C13, C14: value 8p -> 10p; Manufacturer Murata Electronics -> Samsung Electro-Mechanics; Manufacturer Part Number GCM1555C1H8R0FA16D -> CL05C100JB5NNNC
- SW1: Manufacturer DongGuan KINGTEK Industrial Co.,LTD -> SM Switch; Manufacturer Part Number DSIC02LSGET -> SMXS-02K-TP
Connections:
- net GND: now also D3.2, D3.5, J3.3 (Pin_3)
- net NRST: now also D3.4
- net OSC_OUT: now also R8.2; no longer C14.1, X1.3
- net SWCLK: now also D3.3
- net SWDIO: now also D3.1
- net UART_CN_RX: now also J3.2 (Pin_2)
- net UART_CN_TX: now also J3.1 (Pin_1)
- new net: C14.1, R8.1, X1.3
Other:
- note removed: "Power LED"
- moved on the sheet: C13, D2, FID1, FID2, FID3, J2, MH1, MH2, MH3, MH4, R5, U1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
